File: BusinessCard.kicad_pcb (KiCad board)
At the start: 4 copper layers, 89 x 51 mm, 38 parts, among them J1 USB_B, U2 JW5211, U3 JW5211, U4 JW5211, U5 F1C200s, U6 W25Q80DVSNIG, Y1 24MHz

Commit message: progressa
Parts:
- moved C8 15.4 mm to (213.9, 98.4)
- moved R11 15.4 mm to (226.9, 103.4)
- moved R3 15.4 mm to (205.5, 103.6)
- moved U3 15.4 mm to (207.6, 105.0)
- moved C12 15.4 mm to (211.8, 104.9)
- moved C13 15.4 mm to (212.5, 104.1)
- moved C14 15.4 mm to (213.3, 104.9)
- moved C17 15.4 mm to (220.5, 95.5)
- moved C18 15.4 mm to (223.8, 92.2)
- moved C4 15.4 mm to (210.2, 103.5)
- moved C6 15.4 mm to (212.5, 98.4)
- moved C7 15.4 mm to (213.2, 98.4)
- moved C9 15.4 mm to (214.6, 98.4)
- moved L2 15.4 mm to (210.2, 105.4)
- moved R1 15.4 mm to (215.7, 95.3)
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Routing:
- net (no net): track 155.5 -> 0.00 mm

Commit message: progressa
Parts:
- moved C8 15.4 mm to (225.4, 108.7)
- moved R11 15.4 mm to (238.4, 113.7)
- moved R3 15.4 mm to (217.0, 113.9)
- moved U3 15.4 mm to (219.1, 115.3)
- moved C12 15.4 mm to (223.3, 115.2)
- moved C13 15.4 mm to (224.0, 114.4)
- moved C14 15.4 mm to (224.8, 115.2)
- moved C17 15.4 mm to (232.0, 105.8)
- moved C18 15.4 mm to (235.3, 102.5)
- moved C4 15.4 mm to (221.7, 113.8)
- moved C6 15.4 mm to (224.0, 108.7)
- moved C7 15.4 mm to (224.7, 108.7)
- moved C9 15.4 mm to (226.1, 108.7)
- moved L2 15.4 mm to (221.7, 115.7)
- moved R1 15.4 mm to (227.2, 105.6)
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
Commit message: progressa
Routing:
- net (no net): track 0.00 -> 155.5 mm
Changed lines of the file:
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@@
+	)
+	(segment
+		(start 212.7 104.2)
+		(end 212.7 102.7)
+		(width 0.2)
+		(layer "F.Cu")
+		(net 0)
+	)
+	(segment
+		(start 191.8 91.5)
+		(end 227.2 91.5)
+		(width 0.2)
+		(layer "F.Cu")
+		(net 0)
+	)
+	(segment
+		(start 253.9 97.5)
+		(end 253.9 96)
+		(width 0.2)
+		(layer "F.Cu")
+		(net 0)
+	)
+	(segment
+		(start 233.2 97.5)
+		(end 253.9 97.5)
+		(width 0.2)
+		(layer "F.Cu")
+		(net 0)
+	)
+	(segment
+		(start 191.8 93.2)
+		(end 191.8 91.5)
+		(width 0.2)
+		(layer "F.Cu")
+		(net 0)
+	)
+	(segment
+		(start 201.4 102.8)
+		(end 191.8 93.2)
+		(width 0.2)
+		(layer "F.Cu")
+		(net 0)
+	)
+	(segment
+		(start 240.9 93.4)
+		(end 249.9 102.4)
+		(width 0.2)
+		(layer "F.Cu")
+		(net 0)
+	)
+	(segment
+		(start 253.9 96)
+		(end 244.9 87)
+		(width 0.2)
+		(layer "F.Cu")
+		(net 0)
+	)
+	(segment
+		(start 227.2 91.5)
+		(end 228 92.3)
+		(width 0.2)
+		(layer "F.Cu")
+		(net 0)
+	)
+	(segment
+		(start 214.9 93.7)
+		(end 210.5 93.7)
+		(width 0.2)
+		(layer "F.Cu")
+		(net 0)
+	)
+	(segment
+		(start 228 92.3)
+		(end 233.2 97.5)
+		(width 0.2)
+		(layer "F.Cu")
+		(net 0)
+	)
+	(segment
+		(start 234.2 93.4)
+		(end 240.9 93.4)
+		(width 0.2)
+		(layer "F.Cu")
+		(net 0)
+	)
+	(segment
+		(start 244.9 87)
+		(end 240.6 87)
+		(width 0.2)
+		(layer "F.Cu")
+		(net 0)
+	)
+	(segment
+		(start 212.7 102.7)
+		(end 205.7 95.7)
+		(width 0.2)
+		(layer "F.Cu")
+		(net 0)
+	)
+	(segment
+		(start 240.6 87)
+		(end 234.2 93.4)
+		(width 0.2)
+		(layer "F.Cu")
+		(net 0)
+	)
+	(segment
+		(start 210.5 93.7)
+		(end 201.4 102.8)
+		(width 0.2)
+		(layer "F.Cu")
+		(net 0)
 	)
 	(segment
@@
 	)
 	(segment
-		(start 187.452014 107.797986)
-		(end 190.193153 105.056847)
+		(start 191.083384 109.71687)
+		(end 188.87879 111.921464)
 		(width 0.2)
 		(layer "F.Cu")
@@
 	)
 	(segment
-		(start 187.452014 110.494688)
-		(end 187.452014 107.797986)
+		(start 190.193153 105.056847)
+		(end 191.083384 105.947078)
 		(width 0.2)
 		(layer "F.Cu")
@@
 	)
 	(segment
-		(start 188.87879 111.921464)
-		(end 187.452014 110.494688)
-		(width 0.2)
-		(layer "F.Cu")
+		(start 191.083384 105.947078)
+		(end 191.083384 109.71687)
+		(width 0.2)
+		(layer "F.Cu")
