File: BusinessCard.kicad_pcb (KiCad board)
At the start: 2 copper layers, 89 x 51 mm, 39 parts, among them J1 USB_B, U1 JW5211, U2 JW5211, U3 JW5211, U5 F1C200s, U6 W25Q80DVSNIG, Y1 24MHz

Commit message: progressa
Parts:
- moved C6 20.2 mm to (248.8, 110.2)
- moved C7 15.5 mm to (248.9, 108.5), turned to 0 degrees
- moved R11 15.1 mm to (238.0, 114.2), turned to 45 degrees
- moved R12 12.5 mm to (239.0, 113.2), turned to 45 degrees
- moved C14 8.33 mm to (249.0, 113.5), turned to -135 degrees
- moved C13 7.75 mm to (240.8, 109.0), turned to 45 degrees
- moved C17 7.72 mm to (249.0, 103.5)
- moved C16 7.36 mm to (239.3, 107.7), turned to 45 degrees
- moved C9 6.91 mm to (245.8, 114.0), turned to 45 degrees
- moved C12 6.06 mm to (249.2, 107.5), turned to 180 degrees
- moved C10 5.82 mm to (243.0, 114.8), turned to 135 degrees
- moved C15 4.85 mm to (241.8, 106.2), turned to 45 degrees
- moved C8 4.82 mm to (243.0, 110.2), turned to -135 degrees
- moved C11 4.08 mm to (247.8, 112.5), turned to 45 degrees
Connections:
- R12 pad 2: Net-(U5B-AGND) -> GND
- U5 pad 74: Net-(U5B-AGND) -> GND
- U5 pad 82: Net-(U5B-AGND) -> GND
- U5 pad 89: Net-(U5B-AGND) -> GND
Routing:
- net FUSE_PWR: track 14.9 -> 51.7 mm
- net +3V3: track 14.7 -> 8.97 mm, vias 4 -> 1
- net +2V5: track 6.76 -> 7.56 mm

Commit message: progress
Parts:
- moved C11 14.8 mm to (247.6, 97.7)
- moved C12 14.8 mm to (249.0, 92.8)
- moved C14 14.8 mm to (248.8, 98.8)
- moved C17 14.8 mm to (248.8, 88.8)
- moved C18 14.8 mm to (248.8, 87.3)
- moved C6 14.8 mm to (248.6, 95.5)
- moved C7 14.8 mm to (248.8, 93.8)
Changed lines of the file:
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@@
 	(footprint "Capacitor_SMD:C_0201_0603Metric"
 		(layer "F.Cu")
-		(at 249 113.5 -135)
+		(at 248.82 98.75 -135)
 		(descr "Capacitor SMD 0201 (0603 Metric), square (rectangular) end terminal, IPC_7351 nominal, (Body size source: https://www.vishay.com/docs/20052/crcw0201e3.pdf), generated with kicad-footprint-generator")
 		(tags "capacitor")
@@
 	(footprint "Capacitor_SMD:C_0201_0603Metric"
 		(layer "F.Cu")
-		(at 249.155 107.5 180)
+		(at 248.975 92.75 180)
 		(descr "Capacitor SMD 0201 (0603 Metric), square (rectangular) end terminal, IPC_7351 nominal, (Body size source: https://www.vishay.com/docs/20052/crcw0201e3.pdf), generated with kicad-footprint-generator")
 		(tags "capacitor")
@@
 	(footprint "Capacitor_SMD:C_0201_0603Metric"
 		(layer "F.Cu")
-		(at 248.773726 110.226274 -135)
+		(at 248.593726 95.476274 -135)
 		(descr "Capacitor SMD 0201 (0603 Metric), square (rectangular) end terminal, IPC_7351 nominal, (Body size source: https://www.vishay.com/docs/20052/crcw0201e3.pdf), generated with kicad-footprint-generator")
 		(tags "capacitor")
@@
 	(footprint "Capacitor_SMD:C_0201_0603Metric"
 		(layer "F.Cu")
-		(at 247.773726 112.476274 45)
+		(at 247.593726 97.726274 45)
 		(descr "Capacitor SMD 0201 (0603 Metric), square (rectangular) end terminal, IPC_7351 nominal, (Body size source: https://www.vishay.com/docs/20052/crcw0201e3.pdf), generated with kicad-footprint-generator")
 		(tags "capacitor")
@@
 	(footprint "Capacitor_SMD:C_0201_0603Metric"
 		(layer "F.Cu")
-		(at 248.95 102.05)
+		(at 248.77 87.3)
 		(descr "Capacitor SMD 0201 (0603 Metric), square (rectangular) end terminal, IPC_7351 nominal, (Body size source: https://www.vishay.com/docs/20052/crcw0201e3.pdf), generated with kicad-footprint-generator")
 		(tags "capacitor")
@@
 	(footprint "Capacitor_SMD:C_0201_0603Metric"
 		(layer "F.Cu")
-		(at 249 103.5)
+		(at 248.82 88.75)
 		(descr "Capacitor SMD 0201 (0603 Metric), square (rectangular) end terminal, IPC_7351 nominal, (Body size source: https://www.vishay.com/docs/20052/crcw0201e3.pdf), generated with kicad-footprint-generator")
 		(tags "capacitor")
@@
 	(footprint "Capacitor_SMD:C_0201_0603Metric"
 		(layer "F.Cu")
-		(at 248.93 108.5)
+		(at 248.75 93.75)
 		(descr "Capacitor SMD 0201 (0603 Metric), square (rectangular) end terminal, IPC_7351 nominal, (Body size source: https://www.vishay.com/docs/20052/crcw0201e3.pdf), generated with kicad-footprint-generator")
 		(tags "capacitor")

Commit message: progress
Parts:
- moved C11 14.8 mm to (247.8, 112.5)
- moved C12 14.8 mm to (249.2, 107.5)
- moved C14 14.8 mm to (249.0, 113.5)
- moved C17 14.8 mm to (249.0, 103.5)
- moved C18 14.8 mm to (248.9, 102.0)
- moved C6 14.8 mm to (248.8, 110.2)
- moved C7 14.8 mm to (248.9, 108.5)
Changed lines of the file:
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@@
 	(footprint "Capacitor_SMD:C_0201_0603Metric"
 		(layer "F.Cu")
-		(at 248.82 98.75 -135)
+		(at 249 113.5 -135)
 		(descr "Capacitor SMD 0201 (0603 Metric), square (rectangular) end terminal, IPC_7351 nominal, (Body size source: https://www.vishay.com/docs/20052/crcw0201e3.pdf), generated with kicad-footprint-generator")
 		(tags "capacitor")
@@
 	(footprint "Capacitor_SMD:C_0201_0603Metric"
 		(layer "F.Cu")
-		(at 248.975 92.75 180)
+		(at 249.155 107.5 180)
 		(descr "Capacitor SMD 0201 (0603 Metric), square (rectangular) end terminal, IPC_7351 nominal, (Body size source: https://www.vishay.com/docs/20052/crcw0201e3.pdf), generated with kicad-footprint-generator")
 		(tags "capacitor")
@@
 	(footprint "Capacitor_SMD:C_0201_0603Metric"
 		(layer "F.Cu")
-		(at 248.593726 95.476274 -135)
+		(at 248.773726 110.226274 -135)
 		(descr "Capacitor SMD 0201 (0603 Metric), square (rectangular) end terminal, IPC_7351 nominal, (Body size source: https://www.vishay.com/docs/20052/crcw0201e3.pdf), generated with kicad-footprint-generator")
 		(tags "capacitor")
@@
 	(footprint "Capacitor_SMD:C_0201_0603Metric"
 		(layer "F.Cu")
-		(at 247.593726 97.726274 45)
+		(at 247.773726 112.476274 45)
 		(descr "Capacitor SMD 0201 (0603 Metric), square (rectangular) end terminal, IPC_7351 nominal, (Body size source: https://www.vishay.com/docs/20052/crcw0201e3.pdf), generated with kicad-footprint-generator")
 		(tags "capacitor")
@@
 	(footprint "Capacitor_SMD:C_0201_0603Metric"
 		(layer "F.Cu")
-		(at 248.77 87.3)
+		(at 248.95 102.05)
 		(descr "Capacitor SMD 0201 (0603 Metric), square (rectangular) end terminal, IPC_7351 nominal, (Body size source: https://www.vishay.com/docs/20052/crcw0201e3.pdf), generated with kicad-footprint-generator")
 		(tags "capacitor")
@@
 	(footprint "Capacitor_SMD:C_0201_0603Metric"
 		(layer "F.Cu")
-		(at 248.82 88.75)
+		(at 249 103.5)
 		(descr "Capacitor SMD 0201 (0603 Metric), square (rectangular) end terminal, IPC_7351 nominal, (Body size source: https://www.vishay.com/docs/20052/crcw0201e3.pdf), generated with kicad-footprint-generator")
 		(tags "capacitor")
@@
 	(footprint "Capacitor_SMD:C_0201_0603Metric"
 		(layer "F.Cu")
-		(at 248.75 93.75)
+		(at 248.93 108.5)
 		(descr "Capacitor SMD 0201 (0603 Metric), square (rectangular) end terminal, IPC_7351 nominal, (Body size source: https://www.vishay.com/docs/20052/crcw0201e3.pdf), generated with kicad-footprint-generator")
 		(tags "capacitor")

Commit message: progress
Parts:
- moved C14 28.2 mm to (220.8, 113.8)
- moved C9 26.6 mm to (219.2, 112.2)
- moved C17 25.9 mm to (223.2, 105.4), turned to -135 degrees
- moved C11 24.7 mm to (223.4, 116.3)
- moved C18 24.5 mm to (224.5, 104.2), turned to 45 degrees
- moved C10 21.6 mm to (221.4, 114.4), turned to 45 degrees
- moved C6 20.4 mm to (229.7, 117.5), turned to 135 degrees
- moved C8 18.7 mm to (225.1, 104.8)
- moved C7 15.8 mm to (233.9, 113.3), turned to 135 degrees
- moved C12 15.6 mm to (234.5, 112.7), turned to -45 degrees
- moved R1 12.6 mm to (235.1, 109.6), turned to -90 degrees
- moved U6 10.4 mm to (238.3, 108.9), turned to -90 degrees
- moved C13 10.3 mm to (230.9, 106.1)
- moved R11 9.26 mm to (232.0, 107.2), turned to -135 degrees
- moved C15 9.16 mm to (232.9, 108.5), turned to -45 degrees
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Routing:
- net +3V3: track 8.97 -> 65.7 mm, vias 1 -> 5
- net +2V5: track 7.56 -> 51.9 mm, vias 0 -> 3
- net +1V1: track 7.10 -> 44.5 mm, vias 0 -> 4
- net USB_DP: track 0.00 -> 34.7 mm, vias 0 -> 2
- net USB_DN: track 0.00 -> 31.6 mm, vias 0 -> 2
- net GND: track 0.00 -> 29.9 mm, vias 0 -> 3
- net SPI_CS: track 0.00 -> 27.5 mm, vias 0 -> 2
- net SPI_CLK: track 0.00 -> 25.2 mm, vias 0 -> 2
- net SPI_MISO: track 0.00 -> 23.4 mm, vias 0 -> 2
- net SPI_MOSI: track 0.00 -> 23.0 mm, vias 0 -> 2
- net Net-(U5B-SVREF): track 0.00 -> 2.48 mm
