File: BusinessCard.kicad_pcb (KiCad board)
At the start: 2 copper layers, 89 x 51 mm, 39 parts, among them J1 USB_B, U1 JW5211, U2 JW5211, U3 JW5211, U5 F1C200s, U6 W25Q80DVSNIG, Y1 24MHz

Commit message: progress
Parts:
- moved C18 1.90 mm to (225.1, 102.4)
- moved C15 0.41 mm to (233.3, 108.4), turned to 0 degrees
Routing:
- net GND: track 29.9 -> 70.0 mm, vias 3 -> 5
- net +3V3: track 65.7 -> 58.8 mm, vias 5 -> 7
- net CLKN: track 4.50 -> 6.38 mm
- net +2V5: track 51.9 -> 51.3 mm

Commit message: progress
Routing:
- net GND: track 70.0 -> 104.2 mm, vias 5 -> 8

Commit message: progress
Parts:
- moved C12 21.1 mm to (229.2, 92.3)
- moved C15 21.1 mm to (228.0, 88.0)
- moved C7 21.1 mm to (228.6, 92.9)
- moved R1 21.1 mm to (229.8, 89.2)
- moved R12 21.1 mm to (227.8, 86.8)
- moved U6 21.1 mm to (233.0, 88.5)

Commit message: progres
Parts:
- moved C12 21.1 mm to (234.5, 112.7)
- moved C15 21.1 mm to (233.3, 108.4)
- moved C7 21.1 mm to (233.9, 113.3)
- moved R1 21.1 mm to (235.1, 109.6)
- moved R12 21.1 mm to (233.1, 107.2)
- moved U6 21.1 mm to (238.3, 108.9)
