File: untitled.kicad_sch (KiCad schematic)
At the start: 19 parts, among them J1 USB_B, U2 JW5211, U3 JW5211, U4 JW5211

Commit message: data
Parts:
- C1, C2, C3, C4, C5: footprint Capacitor_SMD:CP_Elec_3x5.3 -> Capacitor_SMD:C_0201_0603Metric
- L1, L2, L3: footprint Inductor_SMD:L_6.3x6.3_H3 -> Inductor_SMD:L_0603_1608Metric
Changed lines of the file:
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@@
 			)
 		)
-		(property "Footprint" "Inductor_SMD:L_6.3x6.3_H3"
+		(property "Footprint" "Inductor_SMD:L_0603_1608Metric"
 			(at 157.48 60.96 0)
 			(effects
@@
 			)
 		)
-		(property "Footprint" "Capacitor_SMD:CP_Elec_3x5.3"
+		(property "Footprint" "Capacitor_SMD:C_0201_0603Metric"
 			(at 120.3452 71.12 0)
 			(effects
@@
 			)
 		)
-		(property "Footprint" "Capacitor_SMD:CP_Elec_3x5.3"
+		(property "Footprint" "Capacitor_SMD:C_0201_0603Metric"
 			(at 125.4252 71.12 0)
 			(effects
@@
 			)
 		)
-		(property "Footprint" "Capacitor_SMD:CP_Elec_3x5.3"
+		(property "Footprint" "Capacitor_SMD:C_0201_0603Metric"
 			(at 162.2552 95.25 0)
 			(effects
@@
 			)
 		)
-		(property "Footprint" "Capacitor_SMD:CP_Elec_3x5.3"
+		(property "Footprint" "Capacitor_SMD:C_0201_0603Metric"
 			(at 162.2552 119.38 0)
 			(effects
@@
 			)
 		)
-		(property "Footprint" "Capacitor_SMD:CP_Elec_3x5.3"
+		(property "Footprint" "Capacitor_SMD:C_0201_0603Metric"
 			(at 162.2552 71.12 0)
 			(effects
@@
 			)
 		)
-		(property "Footprint" "Inductor_SMD:L_6.3x6.3_H3"
+		(property "Footprint" "Inductor_SMD:L_0603_1608Metric"
 			(at 157.48 109.22 0)
 			(effects
@@
 			)
 		)
-		(property "Footprint" "Inductor_SMD:L_6.3x6.3_H3"
+		(property "Footprint" "Inductor_SMD:L_0603_1608Metric"
 			(at 157.48 85.09 0)
 			(effects

Commit message: progressa
Parts:
- removed R2, R3: 11k, Resistor_SMD:R_0201_0603Metric, symbol Device:R_US
- removed R4: 10k, Resistor_SMD:R_0201_0603Metric, symbol Device:R_US
- removed R5: 49.9k, Resistor_SMD:R_0201_0603Metric, symbol Device:R_US
- removed R6: 36k, Resistor_SMD:R_0201_0603Metric, symbol Device:R_US
- removed R7: 8.2k, Resistor_SMD:R_0201_0603Metric, symbol Device:R_US
- removed U4: JW5211, Package_TO_SOT_SMD:SOT-23-5, symbol 3340_kicad:JW5211
- added C19: 22uF, symbol Device:C
- added R2: 11k, symbol Device:R
- added R3: 49.9k, symbol Device:R
- added R4: 38k, symbol Device:R
- added R5, R7: 12k, symbol Device:R
- added R6: 10k, symbol Device:R
- added U1: JW5211, Package_TO_SOT_SMD:SOT-23-5, symbol 3340_kicad:JW5211
- C1: value 2.2µF -> 10uF; footprint Capacitor_SMD:C_0201_0603Metric -> (none)
- C2: value 2.2µF -> 22uF; footprint Capacitor_SMD:C_0201_0603Metric -> (none)
- C3, C5: value 22µF -> 10uF; footprint Capacitor_SMD:C_0201_0603Metric -> (none)
- C4: value 22µF -> 22uF; footprint Capacitor_SMD:C_0201_0603Metric -> (none)
- F1: footprint Fuse:Fuse_2920_7451Metric -> Fuse:Fuse_0603_1608Metric
- L1, L2, L3: value 2.2µH -> 1.5uH; footprint Inductor_SMD:L_0603_1608Metric -> (none)
Connections:
- net +1V1: now also C19.2, R6.1; no longer C5.1
- net +2V5: now also C4.2, R4.1; no longer C4.1
- net +3V3: now also C2.2, R3.1; no longer C3.1
- net FUSE_PWR: now also C3.1, C5.1, U1.1 (EN), U1.4 (VIN); no longer C2.1
- net GND: now also C2.1, C4.1, C19.1, R2.1, R5.1, R7.1, U1.2 (GND); no longer C2.2, C4.2
- net at U2.3 (SW): now also L2.1; no longer L1.1
- net at U2.5 (FB): now also R4.2, R5.2
- net at U3.3 (SW): now also L3.1; no longer L2.1
- net at U3.5 (FB): now also R6.2, R7.2
- new net: L1.1, U1.3 (SW)
- new net: R2.2, R3.2, U1.5 (FB)

Commit message: progressa
Parts:
- C1, C19, C2, C3, C4, C5: footprint (none) -> Capacitor_SMD:C_0201_0603Metric
- L1, L2, L3: footprint (none) -> Inductor_SMD:L_0201_0603Metric
- R2, R3, R4, R5, R6, R7: footprint (none) -> Resistor_SMD:R_0201_0603Metric
Changed lines of the file:
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@@
 			)
 		)
-		(property "Footprint" ""
+		(property "Footprint" "Resistor_SMD:R_0201_0603Metric"
 			(at 226.06 147.828 90)
 			(effects
@@
 			)
 		)
-		(property "Footprint" ""
+		(property "Footprint" "Resistor_SMD:R_0201_0603Metric"
 			(at 226.06 110.998 90)
 			(effects
@@
 			)
 		)
-		(property "Footprint" ""
+		(property "Footprint" "Inductor_SMD:L_0201_0603Metric"
 			(at 226.06 132.08 0)
 			(effects
@@
 			)
 		)
-		(property "Footprint" ""
+		(property "Footprint" "Resistor_SMD:R_0201_0603Metric"
 			(at 226.06 140.208 90)
 			(effects
@@
 			)
 		)
-		(property "Footprint" ""
+		(property "Footprint" "Inductor_SMD:L_0201_0603Metric"
 			(at 226.06 73.66 0)
 			(effects
@@
 			)
 		)
-		(property "Footprint" ""
+		(property "Footprint" "Inductor_SMD:L_0201_0603Metric"
 			(at 226.06 102.87 0)
 			(effects
@@
 			)
 		)
-		(property "Footprint" ""
+		(property "Footprint" "Capacitor_SMD:C_0201_0603Metric"
 			(at 192.7352 149.86 0)
 			(effects
@@
 			)
 		)
-		(property "Footprint" ""
+		(property "Footprint" "Resistor_SMD:R_0201_0603Metric"
 			(at 226.06 81.788 90)
 			(effects
@@
 			)
 		)
-		(property "Footprint" ""
+		(property "Footprint" "Capacitor_SMD:C_0201_0603Metric"
 			(at 231.4448 138.43 0)
 			(effects
@@
 			)
 		)
-		(property "Footprint" ""
+		(property "Footprint" "Capacitor_SMD:C_0201_0603Metric"
 			(at 231.4448 80.01 0)
 			(effects
@@
 			)
 		)
-		(property "Footprint" ""
+		(property "Footprint" "Capacitor_SMD:C_0201_0603Metric"
 			(at 192.7352 91.44 0)
 			(effects
@@
 			)
 		)
-		(property "Footprint" ""
+		(property "Footprint" "Resistor_SMD:R_0201_0603Metric"
 			(at 226.06 89.408 90)
 			(effects
@@
 			)
 		)
-		(property "Footprint" ""
+		(property "Footprint" "Capacitor_SMD:C_0201_0603Metric"
 			(at 231.4448 109.22 0)
 			(effects
@@
 			)
 		)
-		(property "Footprint" ""
+		(property "Footprint" "Capacitor_SMD:C_0201_0603Metric"
 			(at 192.7352 120.65 0)
 			(effects
@@
 			)
 		)
-		(property "Footprint" ""
+		(property "Footprint" "Resistor_SMD:R_0201_0603Metric"
 			(at 226.06 118.618 90)
 			(effects
