File: cpu.kicad_sch (KiCad schematic)
At the start: 17 parts, among them U5 F1C200s, Y1 24MHz

Commit message: data
Parts:
- C10, C11, C12, C13, C14, C15, C16, C17, C18, C6, C7, C8, C9: footprint Capacitor_SMD:CP_Elec_3x5.3 -> Capacitor_SMD:C_0201_0603Metric
Changed lines of the file:
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@@
 			)
 		)
-		(property "Footprint" "Capacitor_SMD:CP_Elec_3x5.3"
+		(property "Footprint" "Capacitor_SMD:C_0201_0603Metric"
 			(at 213.36 32.0548 0)
 			(effects
@@
 			)
 		)
-		(property "Footprint" "Capacitor_SMD:CP_Elec_3x5.3"
+		(property "Footprint" "Capacitor_SMD:C_0201_0603Metric"
 			(at 213.36 24.4348 0)
 			(effects
@@
 			)
 		)
-		(property "Footprint" "Capacitor_SMD:CP_Elec_3x5.3"
+		(property "Footprint" "Capacitor_SMD:C_0201_0603Metric"
 			(at 109.22 143.8148 0)
 			(effects
@@
 			)
 		)
-		(property "Footprint" "Capacitor_SMD:CP_Elec_3x5.3"
+		(property "Footprint" "Capacitor_SMD:C_0201_0603Metric"
 			(at 167.64 148.8948 0)
 			(effects
@@
 			)
 		)
-		(property "Footprint" "Capacitor_SMD:CP_Elec_3x5.3"
+		(property "Footprint" "Capacitor_SMD:C_0201_0603Metric"
 			(at 167.64 146.3548 0)
 			(effects
@@
 			)
 		)
-		(property "Footprint" "Capacitor_SMD:CP_Elec_3x5.3"
+		(property "Footprint" "Capacitor_SMD:C_0201_0603Metric"
 			(at 109.22 148.8948 0)
 			(effects
@@
 			)
 		)
-		(property "Footprint" "Capacitor_SMD:CP_Elec_3x5.3"
+		(property "Footprint" "Capacitor_SMD:C_0201_0603Metric"
 			(at 109.22 153.9748 0)
 			(effects
@@
 			)
 		)
-		(property "Footprint" "Capacitor_SMD:CP_Elec_3x5.3"
+		(property "Footprint" "Capacitor_SMD:C_0201_0603Metric"
 			(at 167.64 155.2448 0)
 			(effects
@@
 			)
 		)
-		(property "Footprint" "Capacitor_SMD:CP_Elec_3x5.3"
+		(property "Footprint" "Capacitor_SMD:C_0201_0603Metric"
 			(at 109.22 161.5948 0)
 			(effects
@@
 			)
 		)
-		(property "Footprint" "Capacitor_SMD:CP_Elec_3x5.3"
+		(property "Footprint" "Capacitor_SMD:C_0201_0603Metric"
 			(at 109.22 146.3548 0)
 			(effects
@@
 			)
 		)
-		(property "Footprint" "Capacitor_SMD:CP_Elec_3x5.3"
+		(property "Footprint" "Capacitor_SMD:C_0201_0603Metric"
 			(at 109.22 151.4348 0)
 			(effects
@@
 			)
 		)
-		(property "Footprint" "Capacitor_SMD:CP_Elec_3x5.3"
+		(property "Footprint" "Capacitor_SMD:C_0201_0603Metric"
 			(at 167.64 143.8148 0)
 			(effects
@@
 			)
 		)
-		(property "Footprint" "Capacitor_SMD:CP_Elec_3x5.3"
+		(property "Footprint" "Capacitor_SMD:C_0201_0603Metric"
 			(at 167.64 160.3248 0)
 			(effects

Commit message: progressa
Connections:
- net GND: no longer R12.2, U5.74 (TVGND), U5.82 (AGND), U5.89 (EPAD)
- new net: R12.2, U5.74 (TVGND), U5.82 (AGND), U5.89 (EPAD)

Commit message: progressa
Connections:
- net GND: now also R12.2, U5.74 (TVGND), U5.82 (AGND), U5.89 (EPAD)
Changed lines of the file:
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@@
 	)
 	(junction
+		(at 133.35 177.8)
+		(diameter 0)
+		(color 0 0 0 0)
+	)
+	(junction
 		(at 213.36 29.21)
 		(diameter 0)
@@
 					(unit 1)
 				)
+			)
+		)
+	)
+	(symbol
+		(lib_id "power:GND")
+		(at 133.35 177.8 0)
+		(unit 1)
+		(exclude_from_sim no)
+		(in_bom yes)
+		(on_board yes)
+		(dnp no)
+		(property "Reference" "#PWR027"
+			(at 133.35 184.15 0)
+			(effects
+				(font
+					(size 1.27 1.27)
+				)
+				(hide yes)
+			)
+		)
+		(property "Value" "GND"
+			(at 133.35 181.61 0)
+			(effects
+				(font
+					(size 1.27 1.27)
+				)
+			)
+		)
+		(property "Footprint" ""
+			(at 133.35 177.8 0)
+			(effects
+				(font
+					(size 1.27 1.27)
+				)
+				(hide yes)
+			)
+		)
+		(property "Datasheet" ""
+			(at 133.35 177.8 0)
+			(effects
+				(font
+					(size 1.27 1.27)
+				)
+				(hide yes)
+			)
+		)
+		(property "Description" "Power symbol creates a global label with name \"GND\" , ground"
+			(at 133.35 177.8 0)
+			(effects
+				(font
+					(size 1.27 1.27)
+				)
+				(hide yes)
+			)
+		)
+		(pin "1"
+		)
+		(instances
+			(project "BusinessCard"
+				(path "/c52e2ab9-f991-4723-84f3-4c3609519739/ade188c8-d4ad-412f-be09-98a226951bb3"
+					(reference "#PWR027")
+					(unit 1)
+				)
